File: FSAE_S21_v2.kicad_sch (KiCad schematic)
At the start: 53 parts

Commit message: This is a test
Parts:
- added F?: Fuse (5 A), symbol Device:Fuse
- added J?: MyChron 5 (EXP/PC), symbol Connector:DIN-5
- F?: value Fuse (5 A) -> Fuse (????? A)
Connections:
- net Earth: now also J?.2
- net FAN: no longer U?. (V+)
- net at F?.2, F?.2, K?.7: now also F?.2
- new net: F?.1, J?.5
- new net CAN+Exp: J?.1
- new net CAN-Exp: J?.4
- no-connect marks 69 -> 70

Commit message: Update
Parts:
- added U?: Injector Bank 4, symbol Device:Injector
- U?: value Injector Bank 1 -> Injector Bank 3
Connections:
- net Inj4: now reaches U?.10 (Inj_D)
- net Inj3: now reaches U?.13 (Inj_C)
- no-connect marks 70 -> 68

Commit message: Cleaned stuff up
Connections:
- net FP: now also U?.37 (FP(pump))

Commit message: Updates
Moved megasquirt down a bit/rearranged wires. In the process of shifting some other things around so it looks odd rn.
Connections:
- net GND_Sensor: no longer U?.23 (O2)
- net O2: now also U?.23 (O2)
Other:
- moved on the sheet: U?

Commit message: More cleanup...
Spread things out and adjusted stuff, now just missing where pin 37 on megasquirt goes...
Connections:
- net Earth: now also U?.35 (Spark_E), U?.7 (GND)
- net FAN: no longer K?.5
- net WaterPump: no longer K?.5
- net Inj2: now reaches U?.16 (Inj_B)
- net FP renamed HELP
- no-connect marks 68 -> 67
Other:
- moved on the sheet: U?
