File: FSAE_S21_v2.kicad_sch (KiCad schematic)
At the start: 76 parts

Commit message: idk what i changed this time
Connections:
- new net: F?.1, U?.~ (VCC), U?.~ (VCC), U?.~ (VCC), U?.~ (VCC)
Other:
- title: FSAE S21 Wiring Diagram v1.5 -> FSAE S21 Wiring Diagram v2.1
Changed lines of the file:
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@@
 (kicad_sch (version 20211123) (generator eeschema)
-  (paper "User" 599.999 399.999)
+  (paper "User" 599.999 299.999)
   (title_block
-    (title "FSAE S21 Wiring Diagram v1.5")
-    (date "2021-04-25")
-    (rev "1.5")
+    (title "FSAE S21 Wiring Diagram v2.1")
+    (date "2022-01-14")
+    (rev "2.1")
     (company "Virginia Motorsports")
-    (comment 1 "Updated: Changed various fuse sizes")
-    (comment 2 "Updated: Swapped Relays Power/Ground")
-    (comment 3 "Updated: Removed Cooling Switch")
+    (comment 1 "Updated: Added Wire Colors")
   )
   (bus_alias "Sensor" (members ))
@@
     (effects (font (size 1.27 1.27)) (justify left bottom))
   )
+  (label "GND_Sensor" (at 350.52 228.6 0)
+    (effects (font (size 1.27 1.27)) (justify left bottom))
+  )
   (label "RL_Hall_Effect" (at 495.3 153.67 180)
     (effects (font (size 1.27 1.27)) (justify right bottom))
   )
-  (label "GND_Sensor" (at 350.52 224.79 0)
-    (effects (font (size 1.27 1.27)) (justify left bottom))
-  )
   (label "Inj2" (at 226.06 105.41 180)

Commit message: fixed relay wiring
Parts:
- removed SW?: Fuel/Spark Cutoff Switch, symbol Switch:SW_DPST
Connections:
- net V_CKS: no longer K?.3
- net V_PKS: now also K?.3
- new net: F?.1, U?.~ (VCC), U?.~ (VCC), U?.~ (VCC), U?.~ (VCC)
